Commit message: add fingers to angle-vector

File: jsk_aero_robot/jsk_aero_shop/typeJSK/robots/aero.urdf (robot description, URDF)
Before this commit: robot AeroTypeFCESy, 57 links, 56 joints
Joints:
- joint l_indexbase_joint: limit lower=-3.14159 upper=3.14159 effort=100 velocity=0.5 -> lower=-0.872665 upper=0.872665 effort=100 velocity=0.5
- joint l_thumb_joint: limit lower=-3.14159 upper=3.14159 effort=100 velocity=0.5 -> lower=-0.872665 upper=0.872665 effort=100 velocity=0.5
- joint r_indexbase_joint: limit lower=-3.14159 upper=3.14159 effort=25 velocity=0.5 -> lower=-0.872665 upper=0.872665 effort=25 velocity=0.5
- joint r_thumb_joint: limit lower=-3.14159 upper=3.14159 effort=25 velocity=0.5 -> lower=-0.872665 upper=0.872665 effort=25 velocity=0.5
