Commit message: [jsk_kinova_description] add wrist_camera link

File: jsk_kinova_robot/jsk_kinova_description/robots/gen3_lite_gen3_lite_2f.xacro (robot description, xacro)
@@ -11,3 +11,16 @@
     <xacro:include filename="$(find kortex_description)/robots/kortex_robot.xacro" />
     <xacro:load_robot arm="$(arg arm)" gripper="$(arg gripper)" dof="$(arg dof)" vision="false" sim="$(arg sim)"  prefix="$(arg prefix)" />
+    <link name="kinova_wrist_camera_link">
+      <inertial>
+        <origin xyz="0.0 0.0 0.0" rpy="0 0 0" />
+        <mass value="0.0000000001" />
+        <inertia ixx="0.0000000001" ixy="0.0000000001" ixz="0.0000000001"
+            iyy="0.0000000001" iyz="0.0000000001" izz="0.0000000001" />
+      </inertial>
+    </link>
+    <joint name="kinova_wrist_camera_joint" type="fixed" >
+        <origin rpy="0 0 3.14159265" xyz="-0.0891 0 0.0712" />
+        <parent link="$(arg prefix)upper_wrist_link" />
+        <child link="kinova_wrist_camera_link" />
+    </joint>
 </robot>

Commit message: [jsk_kinova_description] update kinova_wrist_camera position

File: jsk_kinova_robot/jsk_kinova_description/robots/gen3_lite_gen3_lite_2f.xacro (robot description, xacro)
@@ -24,6 +24,6 @@
     </link>
     <joint name="kinova_wrist_camera_joint" type="fixed" >
-        <origin rpy="0 0 3.14159265" xyz="-0.0891 0 0.0712" />
-        <parent link="$(arg prefix)upper_wrist_link" />
+        <origin rpy="3.14159265 -1.57079632 0" xyz="0.05 0.018 0.015" />
+        <parent link="$(arg prefix)gripper_base_link" />
         <child link="kinova_wrist_camera_link" />
     </joint>
