Commit message: [jsk_spotkinova_description] update xacro

File: jsk_spotkinova_robot/jsk_spotkinova_description/robots/jsk_spotkinova.urdf.xacro (robot description, xacro)
@@ -12,5 +12,5 @@
   <joint name="left_gripper_base_fixed" type="fixed">
     <origin rpy="0 0 0" xyz="0.1 0 0" />
-    <parent link="front_rail"/>
+    <parent link="jsk_head_mount_frame"/>
     <child link="$(arg prefix)base_link"/>
   </joint>

Commit message: [jsk_spotkinova_robot][jsk_spotkinova_startup][spotkinovaeus] rename spot-kinova and spot_kinova to spotkinvoa

File: jsk_spotkinova_robot/jsk_spotkinova_description/robots/jsk_spotkinova.urdf.xacro (robot description, xacro)
@@ -9,7 +9,6 @@
   </xacro:include>
   <!-- Transform between spot and kinova -->
-  <!-- The same as jsk_spotkinova_startup/launch/spot_kinova_bringup.launch -->
   <joint name="left_gripper_base_fixed" type="fixed">
-    <origin rpy="0 0 0" xyz="0.1 0 0" />
+    <origin rpy="0 0 0" xyz="0 0 0.03" />
     <parent link="jsk_head_mount_frame"/>
     <child link="$(arg prefix)base_link"/>

Commit message: [jsk_spotkinova_description] update robot model

File: jsk_spotkinova_robot/jsk_spotkinova_description/robots/jsk_spotkinova.urdf.xacro (robot description, xacro)
@@ -15,3 +15,26 @@
   </joint>
   <!-- Back P1 Mount -->
+  <joint name="back_p1_mount_joint_fixed" type="fixed">
+    <origin rpy="0 0 0" xyz="-0.1 0 0.25" />
+    <parent link="body"/>
+    <child link="back_p1_mount_link"/>
+  </joint>
+  <link name="back_p1_mount_link">
+    <inertial>
+      <origin xyz="0 0 0" rpy="0 0 0"/>
+      <mass value="0.0001"/>
+      <inertia ixx="0.0000001" ixy="0.0" ixz="0.0" iyy="0.0000001" iyz="0.0" izz="0.0000001"/>
+    </inertial>
+    <visual>
+      <geometry>
+        <box size="0.5 0.4 0.2" />
+      </geometry>
+      <material name="black"/>
+    </visual>
+    <collision>
+      <geometry>
+        <box size="0.5 0.4 0.2" />
+      </geometry>
+    </collision>
+  </link>
 </robot>
