Commit message: [jsk_spot_description] move insta360 link

File: jsk_spot_robot/jsk_spot_description/robots/jsk_spot.urdf.xacro (robot description, xacro)
@@ -41,5 +41,5 @@
     </link>
     <joint name="jsk_payload_frame_to_insta_360_joint" type="fixed">
-        <origin rpy="0 0 0" xyz="0.1 0 0.5" />
+        <origin rpy="0 0 0" xyz="-0.2 0 0.5" />
         <parent link="jsk_payload_frame" />
         <child link="insta360_link" />
