Commit message: [jsk_panda_startup] delete description about fisheye in dual_panda2.urdf.xacro

File: jsk_panda_robot/panda_eus/models/dual_panda2.urdf.xacro (robot description, xacro)
@@ -200,11 +200,4 @@
     <child link="camera_link"/>
     <origin xyz="-0.22 -0.0 1.46" rpy="0 0.88 0"/>
-  </joint>
-  <!-- create camera frame-->
-  <link name="fisheye_frame" />
-  <joint name="fisheye_fixed_joint" type="fixed">
-    <parent link="dual_arm_base"/>
-    <child link="fisheye_frame"/>
-    <origin xyz="0.07 0 1.9" rpy="0 1.3 0"/>
   </joint>
   <!-- realsense -->
@@ -287,58 +280,4 @@
   <xacro:gazebo_transmission joint_name="left_finger_joint1" />
   <xacro:gazebo_transmission joint_name="left_finger_joint2" />
-  <!-- camera -->
-  <gazebo reference="fisheye_frame">
-    <sensor name="fisheye_camera_sensor" type="wideanglecamera" >
-      <!--pose>${pose}</pose-->
-      <always_on>true</always_on>
-      <update_rate>15</update_rate>
-      <visualize>false</visualize>
-      <camera name="fisheye_camera">
-        <horizontal_fov>3.14</horizontal_fov>
-        <image>
-          <width>2048</width>
-          <height>2048</height>
-          <format>R8G8B8</format>
-        </image>
-        <clip>
-          <near>0.02</near>
-          <far>300</far>
-        </clip>
-        <lens> <!-- for Fisheye -->
-          <!-- type: gnomonical, stereographic, equidistant, equisolid_angle, orthographic, custom -->
-          <!-- More information here: https://en.wikipedia.org/wiki/Fisheye_lens#Mapping_function -->
-          <!--type>equidistant</type-->
-          <type>custom</type>  <!-- manually defined mapping function r = c1*f*fun(theta/c2 + c3) -->
-          <custom_function>
-            <c1>2</c1>
-            <c2>2</c2>
-            <c3>0</c3>
-            <f>0.63661977</f> <!-- ( 2.0 / pi ) -->
-            <fun>id</fun> <!-- one of sin,tan,id -->
-          </custom_function>
-          <!-- if it is set to `true` your horizontal FOV will ramain as defined -->
-          <!-- othervise it depends on lens type and custom function, if there is one -->
-          <scale_to_hfov>false</scale_to_hfov>
-          <cutoff_angle>1.5707</cutoff_angle> <!-- clip everything that is outside of this angle -->
-          <!-- resolution of the cubemap texture, the highter it is - the sharper is your image -->
-          <env_texture_size>2048</env_texture_size>
-        </lens>
-      </camera>
-      <plugin name="camera_controller" filename="libgazebo_ros_camera.so">
-        <alwaysOn>true</alwaysOn>
-        <updateRate>0.0</updateRate><!-- ? -->
-        <cameraName>fisheye_camera</cameraName>
-        <imageTopicName>image_raw</imageTopicName>
-        <cameraInfoTopicName>camera_info</cameraInfoTopicName>
-        <frameName>fisheye_frame</frameName>
-        <hackBaseline>0.07</hackBaseline>
-        <distortionK1>0.0</distortionK1>
-        <distortionK2>0.0</distortionK2>
-        <distortionK3>0.0</distortionK3>
-        <distortionT1>0.0</distortionT1>
-        <distortionT2>0.0</distortionT2>
-      </plugin>
-    </sensor>
-  </gazebo>
   <gazebo>
     <plugin name="gazebo_ros_control" filename="libgazebo_ros_control.so">

Commit message: [panda_eus] delete description about xtion in dual_panda2.urdf.xacro

File: jsk_panda_robot/panda_eus/models/dual_panda2.urdf.xacro (robot description, xacro)
@@ -193,11 +193,4 @@
     <child  link="display"/>
     <origin rpy="0.0 0.2 0.0" xyz="0.0 0.0 1.66"/>
-  </joint>
-  <!-- test xtion frame -->
-  <link name="camera_link" />
-  <joint name="camera_fixed_joint" type="fixed">
-    <parent link="dual_arm_base"/>
-    <child link="camera_link"/>
-    <origin xyz="-0.22 -0.0 1.46" rpy="0 0.88 0"/>
   </joint>
   <!-- realsense -->

Commit message: [panda_eus] add realsense model _d435.urdf.xacro from realsense2_description

File: jsk_panda_robot/panda_eus/models/dual_panda2.urdf.xacro (robot description, xacro)
@@ -242,4 +242,12 @@
     <origin xyz="0 0 0.2" rpy="0 -1.570796327 -0.785398163"/>
   </joint>
+  <!-- handcamera  -->
+  <xacro:include filename="$(find realsense2_description)/urdf/_d435.urdf.xacro" />
+  <xacro:sensor_d435 parent="larm_hand" name="lcamera" use_nominal_extrinsics="true">
+    <origin xyz="0.06 0 0.015" rpy="0 -1.570796326 0"/>
+  </xacro:sensor_d435>
+  <xacro:sensor_d435 parent="rarm_hand" name="rcamera" use_nominal_extrinsics="true">
+    <origin xyz="0.06 0 0.015" rpy="0 -1.570796326 0"/>
+  </xacro:sensor_d435>
   <!-- gazebo -->
   <xacro:macro name="gazebo_transmission" params="joint_name" >

Commit message: [panda_eus] adjust position and angle of mesh model of realsense

File: jsk_panda_robot/panda_eus/models/dual_panda2.urdf.xacro (robot description, xacro)
@@ -195,15 +195,5 @@
   </joint>
   <!-- realsense -->
-  <link name="$(arg arm_id_1)_camera_link" >
-    <!-- <geometry> -->
-    <!--   <mesh filename="../../jsk_panda_accessories/realsense/realsense_with_mount.stl"/> -->
-    <!-- </geometry> -->
-    <inertial>
-      <origin xyz="0.0 0.0 0.0" rpt="0 0 0" />
-      <mass value = "0.005" />
-      <inertia ixx="0.0000000001" ixy="0.0000000001" ixz="0.0000000001"
-    	       iyy="0.0000000001" iyz="0.0000000001" izz="0.0000000001" />
-    </inertial>
-  </link>
+  <link name="$(arg arm_id_1)_camera_link"/>
   <joint name="$(arg arm_id_1)_camera_joint" type="fixed">
     <parent link="$(arg arm_id_1)_link7"/>
@@ -211,15 +201,5 @@
     <origin xyz="0.049497475 -0.02828421 0.12375" rpy="1.57079632 -1.57079632 0.78539816"/>
   </joint>
-  <link name="$(arg arm_id_2)_camera_link" >
-    <!-- <geometry> -->
-    <!--   <mesh filename="../../jsk_panda_accessories/realsense/realsense_with_mount.stl"/> -->
-    <!-- </geometry> -->
-    <inertial>
-      <origin xyz="0.0 0.0 0.0" rpt="0 0 0" />
-      <mass value = "0.005" />
-      <inertia ixx="0.0000000001" ixy="0.0000000001" ixz="0.0000000001"
-    	       iyy="0.0000000001" iyz="0.0000000001" izz="0.0000000001" />
-    </inertial>
-  </link>
+  <link name="$(arg arm_id_2)_camera_link"/>
   <joint name="$(arg arm_id_2)_camera_joint" type="fixed">
     <parent link="$(arg arm_id_2)_link7"/>
@@ -227,4 +207,12 @@
     <origin xyz="0.049497475 -0.02828421 0.12375" rpy="1.57079632 -1.57079632 0.78539816"/>
   </joint>
+  <!-- mesh model of realsense -->
+  <xacro:include filename="$(find realsense2_description)/urdf/_d435.urdf.xacro" />
+  <xacro:sensor_d435 parent="$(arg arm_id_1)_link7" name="rarm_camera_mesh" use_nominal_extrinsics="true">
+    <origin xyz="0.053 -0.007 0.113" rpy="2.356 -1.570796326 0"/>
+  </xacro:sensor_d435>
+  <xacro:sensor_d435 parent="$(arg arm_id_2)_link7" name="larm_camera_mesh" use_nominal_extrinsics="true">
+    <origin xyz="0.053 -0.007 0.113" rpy="2.356 -1.570796326 0"/>
+  </xacro:sensor_d435>
   <!-- eus end effector link -->
   <link name="$(arg arm_id_1)_end_effector" >
@@ -242,12 +230,4 @@
     <origin xyz="0 0 0.2" rpy="0 -1.570796327 -0.785398163"/>
   </joint>
-  <!-- handcamera  -->
-  <xacro:include filename="$(find realsense2_description)/urdf/_d435.urdf.xacro" />
-  <xacro:sensor_d435 parent="larm_hand" name="lcamera" use_nominal_extrinsics="true">
-    <origin xyz="0.06 0 0.015" rpy="0 -1.570796326 0"/>
-  </xacro:sensor_d435>
-  <xacro:sensor_d435 parent="rarm_hand" name="rcamera" use_nominal_extrinsics="true">
-    <origin xyz="0.06 0 0.015" rpy="0 -1.570796326 0"/>
-  </xacro:sensor_d435>
   <!-- gazebo -->
   <xacro:macro name="gazebo_transmission" params="joint_name" >
