Commit message: [jsk_panda_robot] Change camera name: camera -> head_camera

File: jsk_panda_robot/panda_eus/models/dual_panda1.urdf.xacro (robot description, xacro)
@@ -3,9 +3,9 @@
        name="dual_panda" >
   <xacro:include filename="$(find panda_eus)/models/dual_panda.urdf.xacro" />
-  <!-- test xtion frame -->
-  <link name="camera_link" />
-  <joint name="camera_fixed_joint" type="fixed">
+  <!-- head camera -->
+  <link name="head_camera_link" />
+  <joint name="head_camera_fixed_joint" type="fixed">
     <parent link="dual_arm_base"/>
-    <child link="camera_link"/>
+    <child link="head_camera_link" />
     <origin xyz="-0.22 -0.0 1.46" rpy="0 0.88 0"/>
   </joint>

Commit message: [panda_eus] Roughly calibrate head_camera pose

File: jsk_panda_robot/panda_eus/models/dual_panda1.urdf.xacro (robot description, xacro)
@@ -4,9 +4,10 @@
   <xacro:include filename="$(find panda_eus)/models/dual_panda.urdf.xacro" />
   <!-- head camera -->
+  <!-- TODO: intrinsic param calibration -> extrinsic param calibration -->
   <link name="head_camera_link" />
   <joint name="head_camera_fixed_joint" type="fixed">
     <parent link="dual_arm_base"/>
     <child link="head_camera_link" />
-    <origin xyz="-0.22 -0.0 1.46" rpy="0 0.88 0"/>
+    <origin xyz="-0.26 -0.01 1.45" rpy="0 0.38 0" />
   </joint>
   <!-- create camera frame-->
