Commit message: [panda_eus] Add the same end-coords as eus model to URDF

File: jsk_panda_robot/panda_eus/models/dual_panda.urdf.xacro (robot description, xacro)
@@ -202,4 +202,19 @@
     <origin rpy="0.0 0.0 -1.5707963267949" xyz="0.08 0.0 1.505"/>
   </joint-->
+  <!-- eus end effector link -->
+  <link name="$(arg arm_id_1)_end_effector" >
+  </link>
+  <joint name="$(arg arm_id_1)_end_effector_joint" type="fixed">
+    <parent link="$(arg arm_id_1)_link7"/>
+    <child link="$(arg arm_id_1)_end_effector"/>
+    <origin xyz="0 0 0.2" rpy="0 -1.570796327 -0.785398163"/>
+  </joint>
+  <link name="$(arg arm_id_2)_end_effector" >
+  </link>
+  <joint name="$(arg arm_id_2)_end_effector_joint" type="fixed">
+    <parent link="$(arg arm_id_2)_link7"/>
+    <child link="$(arg arm_id_2)_end_effector"/>
+    <origin xyz="0 0 0.2" rpy="0 -1.570796327 -0.785398163"/>
+  </joint>
   <!-- gazebo -->
   <xacro:macro name="gazebo_transmission" params="joint_name" >

Commit message: [panda_eus] delete part of pan_tilt_kinect from dual_panda.urdf.xacro

File: jsk_panda_robot/panda_eus/models/dual_panda.urdf.xacro (robot description, xacro)
@@ -194,12 +194,4 @@
     <origin rpy="0.0 0.2 0.0" xyz="0.0 0.0 1.66"/>
   </joint>
-  <!-- pan_tilt -->
-  <!--xacro:include filename="$(find franka_description)/pan_tilt/pan_tilt_kinect.urdf.xacro" />
-  <xacro:pan_tilt_kinect />
-  <joint name="base_to_head" type="fixed" >
-    <parent link="dual_arm_base" />
-    <child  link="pan_tilt_BASE" />
-    <origin rpy="0.0 0.0 -1.5707963267949" xyz="0.08 0.0 1.505"/>
-  </joint-->
   <!-- eus end effector link -->
   <link name="$(arg arm_id_1)_end_effector" >

Commit message: [jsk_panda_robot] Change dual_panda.urdf.xacro to dual_panda1.urdf.xacro & extract common part of dual_panda*.urdf.xacro as dual_panda.urdf.xacro
As a result, dual_panda.l comes not to include camera link.
But this is not a problem because we usually use TF to get that link pose:
https://github.com/start-jsk/rtmros_tutorials/blob/cd77d440b3753c33292fcb6ab731ef799d29a74c/hironx_tutorial/euslisp/hironxjsk-picking-demo.l#L8-L10
If you want to use camera model inside euslisp like https://github.com/jsk-ros-pkg/jsk_recognition/pull/2549#issuecomment-772349653, you should add dual_panda-utils.l.

File: jsk_panda_robot/panda_eus/models/dual_panda.urdf.xacro (robot description, xacro)
@@ -240,72 +240,4 @@
   <xacro:gazebo_transmission joint_name="left_finger_joint1" />
   <xacro:gazebo_transmission joint_name="left_finger_joint2" />
-  <!-- test xtion frame -->
-  <link name="camera_link" />
-  <joint name="camera_fixed_joint" type="fixed">
-    <parent link="dual_arm_base"/>
-    <child link="camera_link"/>
-    <origin xyz="-0.22 -0.0 1.46" rpy="0 0.88 0"/>
-  </joint>
-  <!-- create camera frame-->
-  <link name="fisheye_frame" />
-  <joint name="fisheye_fixed_joint" type="fixed">
-    <parent link="dual_arm_base"/>
-    <child link="fisheye_frame"/>
-    <origin xyz="0.07 0 1.9" rpy="0 1.3 0"/>
-  </joint>
-  <!-- camera -->
-  <gazebo reference="fisheye_frame">
-    <sensor name="fisheye_camera_sensor" type="wideanglecamera" >
-      <!--pose>${pose}</pose-->
-      <always_on>true</always_on>
-      <update_rate>15</update_rate>
-      <visualize>false</visualize>
-      <camera name="fisheye_camera">
-        <horizontal_fov>3.14</horizontal_fov>
-        <image>
-          <width>2048</width>
-          <height>2048</height>
-          <format>R8G8B8</format>
-        </image>
-        <clip>
-          <near>0.02</near>
-          <far>300</far>
-        </clip>
-        <lens> <!-- for Fisheye -->
-          <!-- type: gnomonical, stereographic, equidistant, equisolid_angle, orthographic, custom -->
-          <!-- More information here: https://en.wikipedia.org/wiki/Fisheye_lens#Mapping_function -->
-          <!--type>equidistant</type-->
-          <type>custom</type>  <!-- manually defined mapping function r = c1*f*fun(theta/c2 + c3) -->
-          <custom_function>
-            <c1>2</c1>
-            <c2>2</c2>
-            <c3>0</c3>
-            <f>0.63661977</f> <!-- ( 2.0 / pi ) -->
-            <fun>id</fun> <!-- one of sin,tan,id -->
-          </custom_function>
-          <!-- if it is set to `true` your horizontal FOV will ramain as defined -->
-          <!-- othervise it depends on lens type and custom function, if there is one -->
-          <scale_to_hfov>false</scale_to_hfov>
-          <cutoff_angle>1.5707</cutoff_angle> <!-- clip everything that is outside of this angle -->
-          <!-- resolution of the cubemap texture, the highter it is - the sharper is your image -->
-          <env_texture_size>2048</env_texture_size>
-        </lens>
-      </camera>
-      <plugin name="camera_controller" filename="libgazebo_ros_camera.so">
-        <alwaysOn>true</alwaysOn>
-        <updateRate>0.0</updateRate><!-- ? -->
-        <cameraName>fisheye_camera</cameraName>
-        <imageTopicName>image_raw</imageTopicName>
-        <cameraInfoTopicName>camera_info</cameraInfoTopicName>
-        <frameName>fisheye_frame</frameName>
-        <hackBaseline>0.07</hackBaseline>
-        <distortionK1>0.0</distortionK1>
-        <distortionK2>0.0</distortionK2>
-        <distortionK3>0.0</distortionK3>
-        <distortionT1>0.0</distortionT1>
-        <distortionT2>0.0</distortionT2>
-      </plugin>
-    </sensor>
-  </gazebo>
   <gazebo>
     <plugin name="gazebo_ros_control" filename="libgazebo_ros_control.so">

File: jsk_panda_robot/panda_eus/models/dual_panda2.urdf.xacro (robot description, xacro)
@@ -2,196 +2,5 @@
 <robot xmlns:xacro="http://www.ros.org/wiki/xacro"
        name="dual_panda" >
-  <!-- panda -->
-  <xacro:include filename="$(find franka_description)/robots/panda_arm.xacro" />
-  <xacro:include filename="$(find franka_description)/robots/hand.xacro"/>
-  <!-- arm -->
-  <xacro:arg name="arm_id_1" default="rarm" />
-  <xacro:arg name="arm_id_2" default="larm" />
-  <!-- test dual arm distance = 0.68 m (2021/03/10)-->
-  <!-- right arm with gripper -->
-  <xacro:panda_arm arm_id="$(arg arm_id_1)" connected_to="fixed_base"  xyz="-0.02 -0.34 0.0" safety_distance="0.03"/>
-  <xacro:hand arm_id="$(arg arm_id_1)" rpy="0 0 ${-pi/4}" connected_to="$(arg arm_id_1)_link8" safety_distance="0.03"/>
-  <!-- left arm with gripper -->
-  <xacro:panda_arm arm_id="$(arg arm_id_2)" connected_to="fixed_base"  xyz="-0.02  0.34 0.0" safety_distance="0.03"/>
-  <xacro:hand arm_id="$(arg arm_id_2)" rpy="0 0 ${-pi/4}" connected_to="$(arg arm_id_2)_link8" safety_distance="0.03"/>
-  <link name="fixed_base" />
-  <link name="dual_arm_base" >
-    <!--
-    <visual>
-      <origin xyz="0 -0.4 0" rpy="1.5707963267949 0.0 0.0" />
-      <geometry>
-        <mesh filename="package://franka_description/meshes/dual_franka_base.dae" scale="0.001 0.001 0.001" />
-      </geometry>
-      <material name="misumi">
-        <color rgba="0.75 0.75 0.75 1.0"/>
-      </material>
-    </visual>
-    <collision>
-      <origin xyz="0 -0.4 0" rpy="1.5707963267949 0.0 0.0" />
-      <geometry>
-        <mesh filename="package://franka_description/meshes/dual_franka_base.dae" scale="0.001 0.001 0.001" />
-      </geometry>
-    </collision>
-    -->
-    <visual>
-      <origin xyz="0.3 0 0.71" />
-      <geometry>
-        <box size="0.6 1.2 0.02" />
-      </geometry>
-      <material name="table">
-        <color rgba="0.7 0.6 0.5 1.0"/>
-      </material>
-    </visual>
-    <collision>
-      <origin xyz="0.3 0 0.71" />
-      <geometry>
-        <box size="0.6 1.2 0.02" />
-      </geometry>
-    </collision>
-    <inertial>
-      <mass value="1000" />
-      <origin rpy="0 0 0" xyz="0.0 0.0 0.2"/>
-      <inertia ixx="10.0" ixy="0.0" ixz="0.0"
-               iyy="10.0" iyz="0.0" izz="10.0" />
-    </inertial>
-  </link>
-  <joint name="base_to_fixed" type="fixed">
-    <parent link="dual_arm_base" />
-    <child  link="fixed_base" />
-    <origin xyz="-0.08 0.0 0.8" rpy="0.0 0.0 0.0" />
-  </joint>
-  <!--link name="table_plane">
-    <visual>
-      <origin xyz="0.3 0 0.01" />
-      <geometry>
-        <box size="0.6 1.2 0.02" />
-      </geometry>
-      <material name="table">
-        <color rgba="0.7 0.6 0.5 1.0"/>
-      </material>
-    </visual>
-    <collision>
-      <origin xyz="0.3 0 0.01" />
-      <geometry>
-        <box size="0.6 1.2 0.02" />
-      </geometry>
-    </collision>
-  </link-->
-  <link name="controller_plane0">
-    <visual>
-      <origin xyz="0.3 0 0.01" />
-      <geometry>
-        <box size="0.6 0.8 0.02" />
-      </geometry>
-      <material name="plane">
-        <color rgba="0.6 0.6 0.6 1.0"/>
-      </material>
-    </visual>
-  </link>
-  <!--link name="controller_plane1">
-    <visual>
-      <origin xyz="0.3 0 0.01" />
-      <geometry>
-        <box size="0.6 0.8 0.02" />
-      </geometry>
-      <material  name="plane" />
-    </visual>
-  </link-->
-  <!--joint name="base_to_table_plane" type="fixed">
-    <parent link="dual_arm_base" />
-    <child  link="table_plane" />
-    <origin xyz="0.0 0.0 0.8" rpy="0.0 0.0 0.0" />
-  </joint-->
-  <joint name="base_to_c_plane0" type="fixed">
-    <parent link="dual_arm_base" />
-    <child  link="controller_plane0" />
-    <origin xyz="0.0 0.0 0.2" rpy="0.0 0.0 0.0" />
-  </joint>
-  <!--joint name="base_to_c_plane1" type="fixed">
-    <parent link="dual_arm_base" />
-    <child  link="controller_plane1" />
-    <origin xyz="0.0 0.0 0.5" rpy="0.0 0.0 0.0" />
-  </joint-->
-  <link name="controller0">
-    <visual>
-      <origin xyz="0.3 0 0.134" />
-      <geometry>
-        <box size="0.475 0.423 0.268" />
-      </geometry>
-      <material name="controller">
-        <color rgba="0.5 0.5 0.6 1.0"/>
-      </material>
-    </visual>
-  </link>
-  <!--link name="controller1">
-    <visual>
-      <origin xyz="0.3 0 0.134" />
-      <geometry>
-        <box size="0.475 0.423 0.268" />
-      </geometry>
-      <material name="controller"/>
-    </visual>
-  </link-->
-  <joint name="base_to_c0" type="fixed">
-    <parent link="dual_arm_base" />
-    <child  link="controller0" />
-    <origin xyz="0.0 0.0 0.22" rpy="0.0 0.0 0.0" />
-  </joint>
-  <!--joint name="base_to_c1" type="fixed">
-    <parent link="dual_arm_base" />
-    <child  link="controller1" />
-    <origin xyz="0.0 0.0 0.52" rpy="0.0 0.0 0.0" />
-  </joint-->
-  <!--link name="dual_arm_booth">
-    <visual>
-      <origin rpy="1.5707963267949 0.0 0.0" xyz="0 -0.75 0"/>
-      <geometry>
-        <mesh filename="package://franka_description/meshes/dual_franka_booth.stl"
-              scale="0.001 0.001 0.001" />
-      </geometry>
-      <material name="misumi">
-        <color rgba="0.75 0.75 0.75 1.0"/>
-      </material>
-    </visual>
-    <collision>
-      <origin rpy="1.5707963267949 0.0 0.0" xyz="0 -0.75 0"/>
-      <geometry>
-        <mesh filename="package://franka_description/meshes/dual_franka_booth.stl"
-              scale="0.001 0.001 0.001" />
-      </geometry>
-    </collision>
-    <inertial>
-      <mass value="1000"/>
-      <origin rpy="0 0 0" xyz="0.0 0.0 0.8"/>
-      <inertia ixx="1.0" ixy="0.0" ixz="0.0" iyy="1.0" iyz="0.0" izz="1.0"/>
-    </inertial>
-  </link>
-  <joint name="base_to_booth" type="fixed">
-    <parent link="dual_arm_base"/>
-    <child link="dual_arm_booth"/>
-    <origin rpy="0.0 0.0 0.0" xyz="-0.11 0.0 0.0"/>
-  </joint-->
-  <link name="display">
-   <visual>
-     <geometry>
-       <!--box size="0.03 0.817 0.342"/--> <!-- 34inch wide -->
-       <box size="0.015 0.165 0.150"/> <!-- 12inch -->
-     </geometry>
-     <material name="Display">
-       <color rgba="0.15 0.15 0.15 1.0"/>
-     </material>
-   </visual>
-   <collision>
-     <geometry>
-       <!--box size="0.03 0.817 0.342"/-->
-       <box size="0.015 0.165 0.150"/> <!-- 12inch -->
-     </geometry>
-   </collision>
-  </link>
-  <joint name="base_to_dispaly" type="fixed">
-    <parent link="dual_arm_base"/>
-    <child  link="display"/>
-    <origin rpy="0.0 0.2 0.0" xyz="0.0 0.0 1.66"/>
-  </joint>
+  <xacro:include filename="$(find panda_eus)/models/dual_panda.urdf.xacro" />
   <!-- realsense -->
   <link name="$(arg arm_id_1)_camera_link"/>
@@ -215,56 +24,3 @@
     <origin xyz="0.053 -0.007 0.113" rpy="2.356 -1.570796326 0"/>
   </xacro:sensor_d435>
-  <!-- eus end effector link -->
-  <link name="$(arg arm_id_1)_end_effector" >
-  </link>
-  <joint name="$(arg arm_id_1)_end_effector_joint" type="fixed">
-    <parent link="$(arg arm_id_1)_link7"/>
-    <child link="$(arg arm_id_1)_end_effector"/>
-    <origin xyz="0 0 0.2" rpy="0 -1.570796327 -0.785398163"/>
-  </joint>
-  <link name="$(arg arm_id_2)_end_effector" >
-  </link>
-  <joint name="$(arg arm_id_2)_end_effector_joint" type="fixed">
-    <parent link="$(arg arm_id_2)_link7"/>
-    <child link="$(arg arm_id_2)_end_effector"/>
-    <origin xyz="0 0 0.2" rpy="0 -1.570796327 -0.785398163"/>
-  </joint>
-  <!-- gazebo -->
-  <xacro:macro name="gazebo_transmission" params="joint_name" >
-    <transmission name="${joint_name}_trans">
-      <type>transmission_interface/SimpleTransmission</type>
-      <joint name="${joint_name}">
-        <hardwareInterface>hardware_interface/VelocityJointInterface</hardwareInterface>
-      </joint>
-      <actuator name="${joint_name}_motor">
-        <hardwareInterface>hardware_interface/VelocityJointInterface</hardwareInterface>
-        <mechanicalReduction>1</mechanicalReduction>
-      </actuator>
-    </transmission>
-  </xacro:macro>
-  <xacro:gazebo_transmission joint_name="right_joint1" />
-  <xacro:gazebo_transmission joint_name="right_joint2" />
-  <xacro:gazebo_transmission joint_name="right_joint3" />
-  <xacro:gazebo_transmission joint_name="right_joint4" />
-  <xacro:gazebo_transmission joint_name="right_joint5" />
-  <xacro:gazebo_transmission joint_name="right_joint6" />
-  <xacro:gazebo_transmission joint_name="right_joint7" />
-  <xacro:gazebo_transmission joint_name="left_joint1" />
-  <xacro:gazebo_transmission joint_name="left_joint2" />
-  <xacro:gazebo_transmission joint_name="left_joint3" />
-  <xacro:gazebo_transmission joint_name="left_joint4" />
-  <xacro:gazebo_transmission joint_name="left_joint5" />
-  <xacro:gazebo_transmission joint_name="left_joint6" />
-  <xacro:gazebo_transmission joint_name="left_joint7" />
-  <xacro:gazebo_transmission joint_name="right_finger_joint1" />
-  <xacro:gazebo_transmission joint_name="right_finger_joint2" />
-  <xacro:gazebo_transmission joint_name="left_finger_joint1" />
-  <xacro:gazebo_transmission joint_name="left_finger_joint2" />
-  <gazebo>
-    <plugin name="gazebo_ros_control" filename="libgazebo_ros_control.so">
-      <!--robotNamespace>/</robotNamespace-->
-      <legacyModeNS>false</legacyModeNS>
-      <robotSimType>gazebo_ros_control/DefaultRobotHWSim</robotSimType>
-    </plugin>
-  </gazebo>
 </robot>
