Commit message: [panda_eus] Update panda model
Previous model originally came from https://github.com/YoheiKakiuchi/franka_ros/blob/add_dual_arm/franka_description/robots/dual_panda_robot.urdf.xacro, which was created before buying real robot.
So some parts were different from real robot.
- Adding display and fisheye camera was never carried out.
- Table is not connected to robot (table position and height may vary from demo to demo).
- Pedestals with control boxes were installed under arms.

File: jsk_panda_robot/panda_eus/models/dual_panda.urdf.xacro (robot description, xacro)
@@ -2,58 +2,16 @@
 <robot xmlns:xacro="http://www.ros.org/wiki/xacro"
        name="dual_panda" >
-  <!-- panda -->
+  <!-- load macros -->
   <xacro:include filename="$(find franka_description)/robots/common/franka_arm.xacro" />
   <xacro:include filename="$(find franka_description)/robots/common/franka_hand.xacro"/>
-  <!-- arm -->
+  <!-- arguments -->
   <xacro:arg name="arm_id_1" default="rarm" />
   <xacro:arg name="arm_id_2" default="larm" />
-  <!-- test dual arm distance = 0.68 m (2021/03/10)-->
-  <!-- right arm with gripper -->
-  <xacro:franka_arm arm_id="$(arg arm_id_1)" connected_to="fixed_base"  xyz="-0.02 -0.34 0.0" safety_distance="0.03" joint_limits="${xacro.load_yaml('$(find franka_description)/robots/panda/joint_limits.yaml')}"/>
-  <xacro:franka_hand arm_id="$(arg arm_id_1)" rpy="0 0 ${-pi/4}" connected_to="$(arg arm_id_1)_link8" safety_distance="0.03"/>
-  <!-- left arm with gripper -->
-  <xacro:franka_arm arm_id="$(arg arm_id_2)" connected_to="fixed_base"  xyz="-0.02  0.34 0.0" safety_distance="0.03" joint_limits="${xacro.load_yaml('$(find franka_description)/robots/panda/joint_limits.yaml')}"/>
-  <xacro:franka_hand arm_id="$(arg arm_id_2)" rpy="0 0 ${-pi/4}" connected_to="$(arg arm_id_2)_link8" safety_distance="0.03"/>
+  <!-- test dual arm distance = 0.68 m (2021/03/10) -->
+  <xacro:arg name="arm_distance" default="0.68" />
+  <xacro:property name="arm_id_1_xyz" value="-0.02 ${$(arg arm_distance)/-2.0} 0.0" />
+  <xacro:property name="arm_id_2_xyz" value="-0.02 ${$(arg arm_distance)/2.0} 0.0" />
+  <link name="dual_arm_base" />
   <link name="fixed_base" />
-  <link name="dual_arm_base" >
-    <!--
-    <visual>
-      <origin xyz="0 -0.4 0" rpy="1.5707963267949 0.0 0.0" />
-      <geometry>
-        <mesh filename="package://franka_description/meshes/dual_franka_base.dae" scale="0.001 0.001 0.001" />
-      </geometry>
-      <material name="misumi">
-        <color rgba="0.75 0.75 0.75 1.0"/>
-      </material>
-    </visual>
-    <collision>
-      <origin xyz="0 -0.4 0" rpy="1.5707963267949 0.0 0.0" />
-      <geometry>
-        <mesh filename="package://franka_description/meshes/dual_franka_base.dae" scale="0.001 0.001 0.001" />
-      </geometry>
-    </collision>
-    -->
-    <visual>
-      <origin xyz="0.3 0 0.71" />
-      <geometry>
-        <box size="0.6 1.2 0.02" />
-      </geometry>
-      <material name="table">
-        <color rgba="0.7 0.6 0.5 1.0"/>
-      </material>
-    </visual>
-    <collision>
-      <origin xyz="0.3 0 0.71" />
-      <geometry>
-        <box size="0.6 1.2 0.02" />
-      </geometry>
-    </collision>
-    <inertial>
-      <mass value="1000" />
-      <origin rpy="0 0 0" xyz="0.0 0.0 0.2"/>
-      <inertia ixx="10.0" ixy="0.0" ixz="0.0"
-               iyy="10.0" iyz="0.0" izz="10.0" />
-    </inertial>
-  </link>
   <joint name="base_to_fixed" type="fixed">
     <parent link="dual_arm_base" />
@@ -61,137 +19,82 @@
     <origin xyz="-0.08 0.0 0.8" rpy="0.0 0.0 0.0" />
   </joint>
-  <!--link name="table_plane">
-    <visual>
-      <origin xyz="0.3 0 0.01" />
-      <geometry>
-        <box size="0.6 1.2 0.02" />
-      </geometry>
-      <material name="table">
-        <color rgba="0.7 0.6 0.5 1.0"/>
-      </material>
-    </visual>
-    <collision>
-      <origin xyz="0.3 0 0.01" />
-      <geometry>
-        <box size="0.6 1.2 0.02" />
-      </geometry>
-    </collision>
-  </link-->
-  <link name="controller_plane0">
-    <visual>
-      <origin xyz="0.3 0 0.01" />
-      <geometry>
-        <box size="0.6 0.8 0.02" />
-      </geometry>
-      <material name="plane">
-        <color rgba="0.6 0.6 0.6 1.0"/>
-      </material>
-    </visual>
-  </link>
-  <!--link name="controller_plane1">
-    <visual>
-      <origin xyz="0.3 0 0.01" />
-      <geometry>
-        <box size="0.6 0.8 0.02" />
-      </geometry>
-      <material  name="plane" />
-    </visual>
-  </link-->
-  <!--joint name="base_to_table_plane" type="fixed">
-    <parent link="dual_arm_base" />
-    <child  link="table_plane" />
-    <origin xyz="0.0 0.0 0.8" rpy="0.0 0.0 0.0" />
-  </joint-->
-  <joint name="base_to_c_plane0" type="fixed">
-    <parent link="dual_arm_base" />
-    <child  link="controller_plane0" />
-    <origin xyz="0.0 0.0 0.2" rpy="0.0 0.0 0.0" />
-  </joint>
-  <!--joint name="base_to_c_plane1" type="fixed">
-    <parent link="dual_arm_base" />
-    <child  link="controller_plane1" />
-    <origin xyz="0.0 0.0 0.5" rpy="0.0 0.0 0.0" />
-  </joint-->
-  <link name="controller0">
-    <visual>
-      <origin xyz="0.3 0 0.134" />
-      <geometry>
-        <box size="0.475 0.423 0.268" />
-      </geometry>
-      <material name="controller">
-        <color rgba="0.5 0.5 0.6 1.0"/>
-      </material>
-    </visual>
-  </link>
-  <!--link name="controller1">
-    <visual>
-      <origin xyz="0.3 0 0.134" />
-      <geometry>
-        <box size="0.475 0.423 0.268" />
-      </geometry>
-      <material name="controller"/>
-    </visual>
-  </link-->
-  <joint name="base_to_c0" type="fixed">
-    <parent link="dual_arm_base" />
-    <child  link="controller0" />
-    <origin xyz="0.0 0.0 0.22" rpy="0.0 0.0 0.0" />
-  </joint>
-  <!--joint name="base_to_c1" type="fixed">
-    <parent link="dual_arm_base" />
-    <child  link="controller1" />
-    <origin xyz="0.0 0.0 0.52" rpy="0.0 0.0 0.0" />
-  </joint-->
-  <!--link name="dual_arm_booth">
-    <visual>
-      <origin rpy="1.5707963267949 0.0 0.0" xyz="0 -0.75 0"/>
-      <geometry>
-        <mesh filename="package://franka_description/meshes/dual_franka_booth.stl"
-              scale="0.001 0.001 0.001" />
-      </geometry>
-      <material name="misumi">
-        <color rgba="0.75 0.75 0.75 1.0"/>
-      </material>
-    </visual>
-    <collision>
-      <origin rpy="1.5707963267949 0.0 0.0" xyz="0 -0.75 0"/>
-      <geometry>
-        <mesh filename="package://franka_description/meshes/dual_franka_booth.stl"
-              scale="0.001 0.001 0.001" />
-      </geometry>
-    </collision>
+  <!-- right arm with gripper -->
+  <xacro:franka_arm arm_id="$(arg arm_id_1)" connected_to="fixed_base"  xyz="${arm_id_1_xyz}" safety_distance="0.03" joint_limits="${xacro.load_yaml('$(find franka_description)/robots/panda/joint_limits.yaml')}"/>
+  <xacro:franka_hand arm_id="$(arg arm_id_1)" rpy="0 0 ${-pi/4}" connected_to="$(arg arm_id_1)_link8" safety_distance="0.03"/>
+  <!-- left arm with gripper -->
+  <xacro:franka_arm arm_id="$(arg arm_id_2)" connected_to="fixed_base"  xyz="${arm_id_2_xyz}" safety_distance="0.03" joint_limits="${xacro.load_yaml('$(find franka_description)/robots/panda/joint_limits.yaml')}"/>
+  <xacro:franka_hand arm_id="$(arg arm_id_2)" rpy="0 0 ${-pi/4}" connected_to="$(arg arm_id_2)_link8" safety_distance="0.03"/>
+  <!-- pedestals -->
+  <xacro:property name="arm_to_pedestal_x" value="-0.0445" />  <!-- Based on pedestal's CAD and panda's footprint (https://www.generationrobots.com/media/panda-franka-emika-datasheet.pdf) -->
+  <xacro:macro name="pedestal" params="arm_id">
+    <link name="${arm_id}_pedestal">
+      <visual>
+        <origin xyz="0.0 0.0 0.0" rpy="0.0 0.0 0.0" />
+        <geometry>
+          <mesh filename="package://panda_eus/meshes/pedestal.stl" scale="0.001 0.001 0.001" />
+        </geometry>
+        <material name="metal">
+          <color rgba="0.75 0.75 0.75 1.0" />
+        </material>
+      </visual>
+      <collision>
+        <origin xyz="0.0 0.0 -0.252" rpy="0.0 0.0 0.0" />
+        <geometry>
+          <cylinder radius="0.115" length="0.504" />
+        </geometry>
+      </collision>
+      <collision>
+        <origin xyz="0.10675 0.0 -0.652" rpy="0.0 0.0 0.0" />
+        <geometry>
+          <box size="0.7135 0.68 0.296" />
+        </geometry>
+      </collision>
+    </link>
+    <joint name="${arm_id}_pedestal_joint" type="fixed">
+      <parent link="${arm_id}_link0" />
+      <child  link="${arm_id}_pedestal" />
+      <origin xyz="${arm_to_pedestal_x} 0.0 0.0" rpy="0.0 0.0 0.0" />
+    </joint>
     <inertial>
-      <mass value="1000"/>
-      <origin rpy="0 0 0" xyz="0.0 0.0 0.8"/>
-      <inertia ixx="1.0" ixy="0.0" ixz="0.0" iyy="1.0" iyz="0.0" izz="1.0"/>
+      <!-- We do not know true inertial parameters -->
+      <mass value="1000" />
+      <origin rpy="0 0 0" xyz="0.0 0.0 -0.4" />
+      <inertia ixx="10.0" ixy="0.0" ixz="0.0"
+               iyy="10.0" iyz="0.0" izz="10.0" />
     </inertial>
-  </link>
-  <joint name="base_to_booth" type="fixed">
-    <parent link="dual_arm_base"/>
-    <child link="dual_arm_booth"/>
-    <origin rpy="0.0 0.0 0.0" xyz="-0.11 0.0 0.0"/>
-  </joint-->
-  <link name="display">
-   <visual>
-     <geometry>
-       <!--box size="0.03 0.817 0.342"/--> <!-- 34inch wide -->
-       <box size="0.015 0.165 0.150"/> <!-- 12inch -->
-     </geometry>
-     <material name="Display">
-       <color rgba="0.15 0.15 0.15 1.0"/>
-     </material>
-   </visual>
-   <collision>
-     <geometry>
-       <!--box size="0.03 0.817 0.342"/-->
-       <box size="0.015 0.165 0.150"/> <!-- 12inch -->
-     </geometry>
-   </collision>
-  </link>
-  <joint name="base_to_dispaly" type="fixed">
-    <parent link="dual_arm_base"/>
-    <child  link="display"/>
-    <origin rpy="0.0 0.2 0.0" xyz="0.0 0.0 1.66"/>
-  </joint>
+  </xacro:macro>
+  <xacro:pedestal arm_id="$(arg arm_id_1)" />
+  <xacro:pedestal arm_id="$(arg arm_id_2)" />
+  <!-- Controls (panda's control box) -->
+  <xacro:property name="pedestal_to_control_xyz" value="0.2715 0.0 -0.5515" />
+  <xacro:macro name="control" params="arm_id">
+    <link name="${arm_id}_control">
+      <visual>
+        <origin xyz="0.0 0.0 0.0" rpy="0.0 0.0 0.0" />
+        <geometry>
+          <box size="0.357 0.444 0.089" />
+        </geometry>
+        <material name="black">
+          <!-- Unable to see in default irtviewer
+          <color rgba="0.0 0.0 0.0 1.0" />
+          -->
+          <color rgba="0.15 0.15 0.15 1.0" />
+        </material>
+      </visual>
+      <collision>
+        <origin xyz="0.0 0.0 0.0" rpy="0.0 0.0 0.0" />
+        <geometry>
+          <box size="0.357 0.444 0.089" />
+        </geometry>
+      </collision>
+    </link>
+    <joint name="${arm_id}_control_joint" type="fixed">
+      <parent link="${arm_id}_pedestal" />
+      <child  link="${arm_id}_control" />
+      <origin xyz="${pedestal_to_control_xyz}" rpy="0.0 0.0 0.0" />
+    </joint>
+  </xacro:macro>
+  <xacro:control arm_id="$(arg arm_id_1)" />
+  <xacro:control arm_id="$(arg arm_id_2)" />
   <!-- eus end effector link -->
   <link name="$(arg arm_id_1)_end_effector" >

File: jsk_panda_robot/panda_eus/models/dual_panda1.urdf.xacro (robot description, xacro)
@@ -11,64 +11,3 @@
     <origin xyz="-0.26 -0.01 1.45" rpy="0 0.38 0" />
   </joint>
-  <!-- create camera frame-->
-  <link name="fisheye_frame" />
-  <joint name="fisheye_fixed_joint" type="fixed">
-    <parent link="dual_arm_base"/>
-    <child link="fisheye_frame"/>
-    <origin xyz="0.07 0 1.9" rpy="0 1.3 0"/>
-  </joint>
-  <!-- camera -->
-  <gazebo reference="fisheye_frame">
-    <sensor name="fisheye_camera_sensor" type="wideanglecamera" >
-      <!--pose>${pose}</pose-->
-      <always_on>true</always_on>
-      <update_rate>15</update_rate>
-      <visualize>false</visualize>
-      <camera name="fisheye_camera">
-        <horizontal_fov>3.14</horizontal_fov>
-        <image>
-          <width>2048</width>
-          <height>2048</height>
-          <format>R8G8B8</format>
-        </image>
-        <clip>
-          <near>0.02</near>
-          <far>300</far>
-        </clip>
-        <lens> <!-- for Fisheye -->
-          <!-- type: gnomonical, stereographic, equidistant, equisolid_angle, orthographic, custom -->
-          <!-- More information here: https://en.wikipedia.org/wiki/Fisheye_lens#Mapping_function -->
-          <!--type>equidistant</type-->
-          <type>custom</type>  <!-- manually defined mapping function r = c1*f*fun(theta/c2 + c3) -->
-          <custom_function>
-            <c1>2</c1>
-            <c2>2</c2>
-            <c3>0</c3>
-            <f>0.63661977</f> <!-- ( 2.0 / pi ) -->
-            <fun>id</fun> <!-- one of sin,tan,id -->
-          </custom_function>
-          <!-- if it is set to `true` your horizontal FOV will ramain as defined -->
-          <!-- othervise it depends on lens type and custom function, if there is one -->
-          <scale_to_hfov>false</scale_to_hfov>
-          <cutoff_angle>1.5707</cutoff_angle> <!-- clip everything that is outside of this angle -->
-          <!-- resolution of the cubemap texture, the highter it is - the sharper is your image -->
-          <env_texture_size>2048</env_texture_size>
-        </lens>
-      </camera>
-      <plugin name="camera_controller" filename="libgazebo_ros_camera.so">
-        <alwaysOn>true</alwaysOn>
-        <updateRate>0.0</updateRate><!-- ? -->
-        <cameraName>fisheye_camera</cameraName>
-        <imageTopicName>image_raw</imageTopicName>
-        <cameraInfoTopicName>camera_info</cameraInfoTopicName>
-        <frameName>fisheye_frame</frameName>
-        <hackBaseline>0.07</hackBaseline>
-        <distortionK1>0.0</distortionK1>
-        <distortionK2>0.0</distortionK2>
-        <distortionK3>0.0</distortionK3>
-        <distortionT1>0.0</distortionT1>
-        <distortionT2>0.0</distortionT2>
-      </plugin>
-    </sensor>
-  </gazebo>
 </robot>

Commit message: [jsk_panda_robot] Delete gazebo settings & fix some typos
They were copied from https://github.com/YoheiKakiuchi/franka_ros/tree/add_dual_arm, which does not match recent panda's gazebo.
And we have no immediate plans to use gazebo.
If you want to implement gazebo afresh, check https://github.com/frankaemika/franka_ros/tree/develop/franka_gazebo and https://github.com/k-okada/jsk_demos/tree/science_animal/science_animal

File: jsk_panda_robot/panda_eus/models/dual_panda.urdf.xacro (robot description, xacro)
@@ -112,41 +112,3 @@
     <origin xyz="0 0 0.2" rpy="0 -1.570796327 -0.785398163"/>
   </joint>
-  <!-- gazebo -->
-  <xacro:macro name="gazebo_transmission" params="joint_name" >
-    <transmission name="${joint_name}_trans">
-      <type>transmission_interface/SimpleTransmission</type>
-      <joint name="${joint_name}">
-        <hardwareInterface>hardware_interface/VelocityJointInterface</hardwareInterface>
-      </joint>
-      <actuator name="${joint_name}_motor">
-        <hardwareInterface>hardware_interface/VelocityJointInterface</hardwareInterface>
-        <mechanicalReduction>1</mechanicalReduction>
-      </actuator>
-    </transmission>
-  </xacro:macro>
-  <xacro:gazebo_transmission joint_name="right_joint1" />
-  <xacro:gazebo_transmission joint_name="right_joint2" />
-  <xacro:gazebo_transmission joint_name="right_joint3" />
-  <xacro:gazebo_transmission joint_name="right_joint4" />
-  <xacro:gazebo_transmission joint_name="right_joint5" />
-  <xacro:gazebo_transmission joint_name="right_joint6" />
-  <xacro:gazebo_transmission joint_name="right_joint7" />
-  <xacro:gazebo_transmission joint_name="left_joint1" />
-  <xacro:gazebo_transmission joint_name="left_joint2" />
-  <xacro:gazebo_transmission joint_name="left_joint3" />
-  <xacro:gazebo_transmission joint_name="left_joint4" />
-  <xacro:gazebo_transmission joint_name="left_joint5" />
-  <xacro:gazebo_transmission joint_name="left_joint6" />
-  <xacro:gazebo_transmission joint_name="left_joint7" />
-  <xacro:gazebo_transmission joint_name="right_finger_joint1" />
-  <xacro:gazebo_transmission joint_name="right_finger_joint2" />
-  <xacro:gazebo_transmission joint_name="left_finger_joint1" />
-  <xacro:gazebo_transmission joint_name="left_finger_joint2" />
-  <gazebo>
-    <plugin name="gazebo_ros_control" filename="libgazebo_ros_control.so">
-      <!--robotNamespace>/</robotNamespace-->
-      <legacyModeNS>false</legacyModeNS>
-      <robotSimType>gazebo_ros_control/DefaultRobotHWSim</robotSimType>
-    </plugin>
-  </gazebo>
 </robot>

Commit message: [panda_eus] Change dual_panda's end-coords to the same as single panda

File: jsk_panda_robot/panda_eus/models/dual_panda.urdf.xacro (robot description, xacro)
@@ -101,14 +101,14 @@
   </link>
   <joint name="$(arg arm_id_1)_end_effector_joint" type="fixed">
-    <parent link="$(arg arm_id_1)_link7"/>
+    <parent link="$(arg arm_id_1)_link8"/>
     <child link="$(arg arm_id_1)_end_effector"/>
-    <origin xyz="0 0 0.2" rpy="0 -1.570796327 -0.785398163"/>
+    <origin xyz="0 0 0.1" rpy="0 -1.570796327 -0.785398163"/>
   </joint>
   <link name="$(arg arm_id_2)_end_effector" >
   </link>
   <joint name="$(arg arm_id_2)_end_effector_joint" type="fixed">
-    <parent link="$(arg arm_id_2)_link7"/>
+    <parent link="$(arg arm_id_2)_link8"/>
     <child link="$(arg arm_id_2)_end_effector"/>
-    <origin xyz="0 0 0.2" rpy="0 -1.570796327 -0.785398163"/>
+    <origin xyz="0 0 0.1" rpy="0 -1.570796327 -0.785398163"/>
   </joint>
 </robot>

Commit message: [panda_eus] Move end-coords of single panda and dual_panda to the center of the fingers

File: jsk_panda_robot/panda_eus/models/dual_panda.urdf.xacro (robot description, xacro)
@@ -101,14 +101,14 @@
   </link>
   <joint name="$(arg arm_id_1)_end_effector_joint" type="fixed">
-    <parent link="$(arg arm_id_1)_link8"/>
+    <parent link="$(arg arm_id_1)_hand_tcp"/>
     <child link="$(arg arm_id_1)_end_effector"/>
-    <origin xyz="0 0 0.1" rpy="0 -1.570796327 -0.785398163"/>
+    <origin xyz="0 0 0" rpy="0 -1.570796327 0"/>
   </joint>
   <link name="$(arg arm_id_2)_end_effector" >
   </link>
   <joint name="$(arg arm_id_2)_end_effector_joint" type="fixed">
-    <parent link="$(arg arm_id_2)_link8"/>
+    <parent link="$(arg arm_id_2)_hand_tcp"/>
     <child link="$(arg arm_id_2)_end_effector"/>
-    <origin xyz="0 0 0.1" rpy="0 -1.570796327 -0.785398163"/>
+    <origin xyz="0 0 0" rpy="0 -1.570796327 0"/>
   </joint>
 </robot>

Commit message: [panda_eus] Make URDF follow euslisp model

File: jsk_panda_robot/panda_eus/models/dual_panda.urdf.xacro (robot description, xacro)
@@ -101,14 +101,14 @@
   </link>
   <joint name="$(arg arm_id_1)_end_effector_joint" type="fixed">
-    <parent link="$(arg arm_id_1)_hand_tcp"/>
+    <parent link="$(arg arm_id_1)_hand"/>
     <child link="$(arg arm_id_1)_end_effector"/>
-    <origin xyz="0 0 0" rpy="0 -1.570796327 0"/>
+    <origin xyz="0 0 0.1034" rpy="0 -1.570796327 0"/>
   </joint>
   <link name="$(arg arm_id_2)_end_effector" >
   </link>
   <joint name="$(arg arm_id_2)_end_effector_joint" type="fixed">
-    <parent link="$(arg arm_id_2)_hand_tcp"/>
+    <parent link="$(arg arm_id_2)_hand"/>
     <child link="$(arg arm_id_2)_end_effector"/>
-    <origin xyz="0 0 0" rpy="0 -1.570796327 0"/>
+    <origin xyz="0 0 0.1034" rpy="0 -1.570796327 0"/>
   </joint>
 </robot>

Commit message: add single panda (#1799)
* add single panda

* update from latest franka_control.launch

* add comments

* remove unused config

* remove gazebo descriptions

* move code for panda.l and modify messages

* change name

* change to include franka_control.launch

* change larm to rarm

* panda.urdf.xacro is unnecessary

* [panda_eus] Add panda.urdf and panda.l to .gitignore

* [panda_eus] Extract common part of panda-interface.l and dual_panda-interface.l as panda-common-interface.l

* [jsk_panda_robot] Add single panda to README

* [jsk_panda_robot] Add notice about end-coords, reset-pose, and reset-manip-pose

* [panda_eus] Improve error message from :set-joint-pd-gain

* enable access to gripper-grasp-action

* add missing bracket

* Enable to get results of :stop-gripper/:homing-gripper/:start-grasp/:stop-grasp/:move-gripper from their return values

* Enable to get results of :stop-gripper/:homing-gripper/:start-grasp/:stop-grasp/:move-gripper from separated methods

* Consider compatibility with FR3 (Franka Research 3)

* Remove unnecessary method

* extract action from hash

* Revert "extract action from hash"

This reverts commit 0066eb7ea240d2471c1f17d89b9bb000225caed9.

* Make errors from :get-*-result readable when * is not called

* Force to call all :wait-for-result and postprocess even if some of them fail

* [panda_eus] Change dual_panda's end-coords to the same as single panda

* [panda_eus] Move end-coords of single panda and dual_panda to the center of the fingers

* [panda_eus] Make :gripper method work

* [panda_eus] Make URDF follow euslisp model

* [panda_eus] Enable to get gripper method result without waiting

* [panda_eus] Enable to get status of gripper actions

---------

Co-authored-by: Shun Hasegawa <pazeshun3684@gmail.com>

File: jsk_panda_robot/panda_eus/models/dual_panda.urdf.xacro (robot description, xacro)
@@ -101,14 +101,14 @@
   </link>
   <joint name="$(arg arm_id_1)_end_effector_joint" type="fixed">
-    <parent link="$(arg arm_id_1)_link7"/>
+    <parent link="$(arg arm_id_1)_hand"/>
     <child link="$(arg arm_id_1)_end_effector"/>
-    <origin xyz="0 0 0.2" rpy="0 -1.570796327 -0.785398163"/>
+    <origin xyz="0 0 0.1034" rpy="0 -1.570796327 0"/>
   </joint>
   <link name="$(arg arm_id_2)_end_effector" >
   </link>
   <joint name="$(arg arm_id_2)_end_effector_joint" type="fixed">
-    <parent link="$(arg arm_id_2)_link7"/>
+    <parent link="$(arg arm_id_2)_hand"/>
     <child link="$(arg arm_id_2)_end_effector"/>
-    <origin xyz="0 0 0.2" rpy="0 -1.570796327 -0.785398163"/>
+    <origin xyz="0 0 0.1034" rpy="0 -1.570796327 0"/>
   </joint>
 </robot>
