Commit message: [jsk_fetch_startup] fix parameters of finger_tip.urdf.xacro

File: jsk_fetch_robot/jsk_fetch_startup/robots/finger_tip.urdf.xacro (robot description, xacro)
@@ -30,5 +30,5 @@
     </link>
     <joint name="l_gripper_finger_tip_joint" type="fixed">
-        <origin rpy="0 0 0" xyz="0 0 0" />
+        <origin rpy="0 0 0" xyz="0 -0.001 -0.013" />
         <parent link="l_gripper_finger_link" />
         <child link="l_gripper_finger_tip" />
@@ -64,5 +64,5 @@
     </link>
     <joint name="r_gripper_finger_tip_joint" type="fixed">
-        <origin rpy="3.141592 0 0" xyz="0 0 0" />
+        <origin rpy="3.141592 0 0" xyz="0 0.001 0.013" />
         <parent link="r_gripper_finger_link" />
         <child link="r_gripper_finger_tip" />
